File: design/receiver/receiver.kicad_sch (KiCad schematic)
At the start: 11 parts, among them J3 RCA, U1 LM318N

Commit message: 75 ohm resistor included
Parts:
- R3: now fitted
Changed lines of the file:
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@@
 		(in_bom yes)
 		(on_board yes)
-		(dnp yes)
+		(dnp no)
 		(property "Reference" "R3"
 			(at 93.98 76.2 90)
